Commit message: respond to review comments, fix pixel logic launch file and joints

File: pluto-project-2/my_robot/urdf/my_robot.xacro (robot description, xacro)
@@ -170,6 +170,6 @@
     <axis xyz="0 1 0" rpy="0 0 0"/>
   </joint>
-  <joint type="fixed" name="lidar_joint">
-    <origin xyz=".02 0 0" rpy="0 0 0"/>
+  <joint type="fixed" name="hokuyo_joint">
+    <origin xyz="0.15 0 0.1" rpy="0 0 0"/>
     <child link="hokuyo"/>
     <parent link="chassis"/>
